File: electronics/motor_driver_tmc6300/motor_driver_tmc6300.kicad_pcb (KiCad board)
At the start: 2 copper layers, 30.5 x 30.5 mm, 73 parts, among them IC1 TMC6300, U1 U, U2 U, U3 U, U4 U

Commit message: update
Parts:
- removed kibuzzard-6702242B (x2): G***, kibuzzard-6702242B
- removed kibuzzard-670235E4 (x2): G***, kibuzzard-670235E4
- added TP1: TestPoint, Library:kawashima_TestPoint_THTPad_D1.5mm_Drill0.7mm, F.Cu at (120.7, 109.2)
- added TP2: TestPoint, Library:kawashima_TestPoint_THTPad_D1.5mm_Drill0.7mm, F.Cu at (123.2, 111.8)
- added TP3: TestPoint, Library:kawashima_TestPoint_THTPad_D1.5mm_Drill0.7mm, F.Cu at (120.7, 111.8)
- added TP4: TestPoint, Library:kawashima_TestPoint_THTPad_D1.5mm_Drill0.7mm, F.Cu at (123.2, 109.2)
- added kibuzzard-67032619: G***, kibuzzard-67032619, F.Cu at (123.2, 115.1)
- added kibuzzard-67032626: G***, kibuzzard-67032626, F.Cu at (125.7, 114.7)
- moved TMC_DIAG1 5.21 mm to (125.9, 109.2)
- moved TMC_DIAG2 5.21 mm to (125.9, 111.8)
Connections:
- IC1 pad 16: GND -> Net-(IC1-BRUV)
- IC1 pad 20: GND -> Net-(IC1-BRW)
Routing:
- net +3V3: track 74.4 -> 96.1 mm
- net Net-(IC1-BRW): track 0.00 -> 17.1 mm, vias 0 -> 1
- net Net-(IC1-BRUV): track 0.00 -> 14.3 mm, vias 0 -> 1
- net /TMC_DIAG: track 15.1 -> 12.7 mm
- net +5V: track 76.1 -> 74.4 mm
- net Net-(IC1-V): vias 0 -> 1
- net Net-(IC1-W): vias 0 -> 1
- net Net-(IC1-U): vias 0 -> 1
- net GND: vias 73 -> 111
- net (no net): vias 1 -> 0
- added copper zone on B.Cu, net Net-(IC1-BRUV)
- added copper zone on F.Cu, net Net-(IC1-BRUV)
- added copper zone on B.Cu, net Net-(IC1-BRW)
- added copper zone on F.Cu, net Net-(IC1-BRW)
Other:
- board text added: "5V"
